File: Ragnohacks PCB.kicad_sch (KiCad schematic)
At the start: 35 parts, among them J1 Conn_01x02, J2 Conn_01x18, J3 Conn_01x18, J4 USB_A, SW1 SW_Push, U1 RP2040, U2 W25Q128JVS, U3 LD1117S33TR_SOT223, U4 USBLC6-2P6, Y1 12MHz

Commit message: Finish schematic and part choosing, get initial quote
Parts:
- D1, D3: LCSC (none) -> C965804; LSCS C965804 -> (none)
- D2: LCSC (none) -> C2480; LSCS C2480 -> (none)
- J1: footprint Connector_PinHeader_2.54mm:PinHeader_1x02_P2.54mm_Horizontal -> Connector_PinHeader_2.54mm:PinHeader_1x02_P2.54mm_Vertical; LCSC (none) -> C7501612; LSCS C7501612 -> (none)
- J2, J3: footprint Connector_PinSocket_2.54mm:PinSocket_1x18_P2.54mm_Horizontal -> Connector_PinSocket_2.54mm:PinSocket_1x18_P2.54mm_Vertical; LCSC (none) -> C2897400; LSCS C2897400 -> (none)
- J4: LCSC (none) -> C319178; LSCS C319178 -> (none)
- R3, R4: value 460R -> 360R; footprint Resistor_SMD:R_0402_1005Metric -> Resistor_SMD:R_0603_1608Metric
- SW1: footprint Button_Switch_SMD:SW_Push_1P1T_NO_6x6mm_H9.5mm -> Button_Switch_SMD:SW_Push_1P1T_XKB_TS-1187A; LCSC (none) -> C318884; LSCS C500080 -> (none)
- U1: LCSC (none) -> C2040; LSCS C2040 -> (none)
- U2: LCSC (none) -> W25Q128JVSIQ; LSCS W25Q128JVSIQ -> (none)
- U3: LCSC (none) -> C35879; LSCS C35879 -> (none)
- U4: LCSC (none) -> C2682291; LSCS C2682291 -> (none)
- Y1: LCSC (none) -> C18209050; LSCS C18209050 -> (none)
Changed lines of the file:
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@@
 			)
 		)
-		(property "LSCS" "C2682291"
+		(property "LCSC" "C2682291"
 			(at 58.42 162.56 0)
 			(effects
@@
 			)
 		)
-		(property "LSCS" ""
+		(property "LCSC" ""
 			(at 170.18 27.94 0)
 			(effects
@@
 			)
 		)
-		(property "LSCS" ""
+		(property "LCSC" ""
 			(at 182.88 27.94 0)
 			(effects
@@
 			)
 		)
+		(property "LCSC" ""
+			(at 43.18 105.41 0)
+			(effects
+				(font
+					(size 1.27 1.27)
+				)
+				(hide yes)
+			)
+		)
 		(pin "1"
 		)
@@
 			)
 		)
-		(property "Value" "460R"
+		(property "Value" "360R"
 			(at 123.19 163.8299 0)
 			(effects
@@
 			)
 		)
-		(property "Footprint" "Resistor_SMD:R_0402_1005Metric"
+		(property "Footprint" "Resistor_SMD:R_0603_1608Metric"
 			(at 118.872 162.56 90)
 			(effects
@@
 			)
 		)
+		(property "LCSC" ""
+			(at 120.65 162.56 0)
+			(effects
+				(font
+					(size 1.27 1.27)
+				)
+				(hide yes)
+			)
+		)
 		(pin "1"
 		)
@@
 			)
 		)
-		(property "LSCS" ""
+		(property "LCSC" ""
 			(at 53.34 29.21 0)
 			(effects
@@
 			)
 		)
-		(property "Footprint" "Button_Switch_SMD:SW_Push_1P1T_NO_6x6mm_H9.5mm"
+		(property "Footprint" "Button_Switch_SMD:SW_Push_1P1T_XKB_TS-1187A"
 			(at 25.4 44.45 0)
 			(effects
@@
 			)
 		)
-		(property "LSCS" "C500080"
+		(property "LCSC" "C318884"
 			(at 25.4 49.53 0)
 			(effects
@@
 			)
 		)
-		(property "Footprint" "Connector_PinHeader_2.54mm:PinHeader_1x02_P2.54mm_Horizontal"
+		(property "Footprint" "Connector_PinHeader_2.54mm:PinHeader_1x02_P2.54mm_Vertical"
 			(at 40.64 115.57 0)
 			(effects
@@
 			)
 		)
-		(property "LSCS" "C7501612"
+		(property "LCSC" "C7501612"
 			(at 40.64 115.57 0)
 			(effects
@@
 			)
 		)
-		(property "Value" "460R"
+		(property "Value" "360R"
 			(at 146.05 128.2699 0)
 			(effects
@@
 			)
 		)
-		(property "Footprint" "Resistor_SMD:R_0402_1005Metric"
+		(property "Footprint" "Resistor_SMD:R_0603_1608Metric"
 			(at 141.732 127 90)
 			(effects
@@
 			)
 		)
+		(property "LCSC" ""
+			(at 143.51 127 0)
+			(effects
+				(font
+					(size 1.27 1.27)
+				)
+				(hide yes)
+			)
+		)
 		(pin "1"
 		)
@@
 			)
 		)
-		(property "LSCS" ""
+		(property "LCSC" ""
 			(at 66.04 29.21 0)
 			(effects
@@
 			)
 		)
-		(property "LSCS" ""
+		(property "LCSC" ""
 			(at 106.68 27.94 0)
 			(effects
@@
 			)
 		)
-		(property "LSCS" ""
+		(property "LCSC" ""
 			(at 93.98 27.94 0)
 			(effects
@@
 			)
 		)
-		(property "LSCS" ""
+		(property "LCSC" ""
 			(at 25.4 106.68 0)
 			(effects
@@
 			)
 		)
-		(property "LSCS" "C2480"
+		(property "LCSC" "C2480"
 			(at 48.26 153.67 0)
 			(effects
@@
 			)
 		)
-		(property "LSCS" ""
+		(property "LCSC" ""
 			(at 107.95 153.67 0)
 			(effects
@@
 			)
 		)
+		(property "LCSC" ""
+			(at 43.18 45.72 0)
+			(effects
+				(font
+					(size 1.27 1.27)
+				)
+				(hide yes)
+			)
+		)
 		(pin "1"
 		)
@@
 			)
 		)
-		(property "LSCS" ""
+		(property "LCSC" ""
 			(at 40.64 29.21 0)
 			(effects
@@
 			)
 		)
-		(property "LSCS" ""
+		(property "LCSC" ""
 			(at 25.4 92.71 0)
 			(effects
@@
 			)
 		)
-		(property "LSCS" "C965804"
+		(property "LCSC" "C965804"
 			(at 120.65 153.67 0)
 			(effects
@@
 			)
 		)
-		(property "LSCS" ""
+		(property "LCSC" ""
 			(at 132.08 27.94 0)
 			(effects
@@
 			)
 		)
-		(property "LSCS" ""
+		(property "LCSC" ""
 			(at 25.4 54.61 0)
 			(effects
@@
 			)
 		)
-		(property "LSCS" ""
+		(property "LCSC" ""
 			(at 73.66 153.67 0)
 			(effects
@@
 			)
 		)
-		(property "LSCS" "C2040"
+		(property "LCSC" "C2040"
 			(at 78.74 87.63 0)
 			(effects
@@
 			)
 		)
-		(property "LSCS" ""
+		(property "LCSC" ""
 			(at 144.78 27.94 0)
 			(effects
@@
 			)
 		)
-		(property "LSCS" "C319178"
+		(property "LCSC" "C319178"
 			(at 36.83 162.56 0)
 			(effects
@@
 			)
 		)
-		(property "LSCS" "C965804"
+		(property "LCSC" "C965804"
 			(at 143.51 118.11 0)
 			(effects
@@
 			)
 		)
-		(property "LSCS" ""
+		(property "LCSC" ""
 			(at 179.07 63.5 0)
 			(effects
@@
 			)
 		)
-		(property "LSCS" "C18209050"
+		(property "LCSC" "C18209050"
 			(at 29.21 100.33 0)
 			(effects
@@
 			)
 		)
-		(property "LSCS" "C35879"
+		(property "LCSC" "C35879"
 			(at 87.63 149.86 0)
 			(effects
@@
 			)
 		)
-		(property "LSCS" ""
+		(property "LCSC" ""
 			(at 195.58 27.94 0)
 			(effects
@@
 			)
 		)
-		(property "LSCS" ""
+		(property "LCSC" ""
 			(at 157.48 27.94 0)
 			(effects
@@
 			)
 		)
-		(property "LSCS" ""
+		(property "LCSC" ""
 			(at 119.38 27.94 0)
 			(effects
@@
 			)
 		)
-		(property "Footprint" "Connector_PinSocket_2.54mm:PinSocket_1x18_P2.54mm_Horizontal"
+		(property "Footprint" "Connector_PinSocket_2.54mm:PinSocket_1x18_P2.54mm_Vertical"
 			(at 196.85 127 0)
 			(effects
@@
 			)
 		)
-		(property "LSCS" "C2897400"
+		(property "LCSC" "C2897400"
 			(at 196.85 127 0)
 			(effects
@@
 			)
 		)
-		(property "Footprint" "Connector_PinSocket_2.54mm:PinSocket_1x18_P2.54mm_Horizontal"
+		(property "Footprint" "Connector_PinSocket_2.54mm:PinSocket_1x18_P2.54mm_Vertical"
 			(at 193.04 127 0)
 			(effects
@@
 			)
 		)
-		(property "LSCS" "C2897400"
+		(property "LCSC" "C2897400"
 			(at 193.04 127 0)
 			(effects
@@
 			)
 		)
-		(property "LSCS" "W25Q128JVSIQ"
+		(property "LCSC" "W25Q128JVSIQ"
 			(at 166.37 73.66 0)
 			(effects

Commit message: Start layout, add PCBWay parts
Parts:
- C1, C11, C12, C15, C16, C17, C2, C3, C4, C5, C6, C7, C8: MPN (none) -> CL05B104KP5NNNC
- C10, C9: MPN (none) -> CL05A105KO5NNNC
- C13, C14: value 24pF -> 18pF; MPN (none) -> GRM1555C1H180JA01D
- C18: MPN (none) -> GRM155R60J106ME05D
- D1, D3: MPN (none) -> 150060GS75000
- D2: MPN (none) -> SK12
- J1: MPN (none) -> 10129379-902002BLF
- J2, J3: MPN (none) -> PPPC181LGBN-RC
- J4: MPN (none) -> 931
- R1: MPN (none) -> D1TFAS0402R1001F-T10
- R2: MPN (none) -> D1TFA0402R1002F-T10
- R3, R4: footprint Resistor_SMD:R_0603_1608Metric -> Resistor_SMD:R_0402_1005Metric; MPN (none) -> RC0402FR-13360RL
- SW1: MPN (none) -> PTS645SK43SMTR92 LFS
- U1: MPN (none) -> SC0914(13)
- U2: MPN (none) -> W25Q128JVSIQ
- U3: MPN (none) -> LD1117S33TR
- U4: MPN (none) -> USBLC6-2P6
- Y1: MPN (none) -> RH100-12.000-12-1010-X-TR-NS2
Connections:
- net A0: now also U1.41 (GPIO29_ADC3); no longer U1.38 (GPIO26_ADC0)
- net A1: now also U1.40 (GPIO28_ADC2); no longer U1.39 (GPIO27_ADC1)
- net A2: now also U1.39 (GPIO27_ADC1); no longer U1.40 (GPIO28_ADC2)
- net A3: now also U1.38 (GPIO26_ADC0); no longer U1.41 (GPIO29_ADC3)
- net D0: now also U1.37 (GPIO25); no longer U1.2 (GPIO0)
- net D1: now also U1.36 (GPIO24); no longer U1.3 (GPIO1)
- net D10: now also U1.18 (GPIO15); no longer U1.13 (GPIO10)
- net D11: now also U1.17 (GPIO14); no longer U1.14 (GPIO11)
- net D12: now also U1.16 (GPIO13); no longer U1.15 (GPIO12)
- net D13: now also U1.15 (GPIO12); no longer U1.16 (GPIO13)
- net D14: now also U1.14 (GPIO11); no longer U1.17 (GPIO14)
- net D15: now also U1.13 (GPIO10); no longer U1.18 (GPIO15)
- net D16: now also U1.12 (GPIO9); no longer U1.27 (GPIO16)
- net D17: now also U1.11 (GPIO8); no longer U1.28 (GPIO17)
- net D18: now also U1.9 (GPIO7); no longer U1.29 (GPIO18)
- net D19: now also U1.8 (GPIO6); no longer U1.30 (GPIO19)
- net D2: now also U1.35 (GPIO23); no longer U1.4 (GPIO2)
- net D20: now also U1.7 (GPIO5); no longer U1.31 (GPIO20)
- net D21: now also U1.6 (GPIO4); no longer U1.32 (GPIO21)
- net D22: now also U1.5 (GPIO3); no longer U1.34 (GPIO22)
- net D23: now also U1.4 (GPIO2); no longer U1.35 (GPIO23)
- net D24: now also U1.3 (GPIO1); no longer U1.36 (GPIO24)
- net D3: now also U1.34 (GPIO22); no longer U1.5 (GPIO3)
- net D4: now also U1.32 (GPIO21); no longer U1.6 (GPIO4)
- net D5: now also U1.31 (GPIO20); no longer U1.7 (GPIO5)
- net D6: now also U1.30 (GPIO19); no longer U1.8 (GPIO6)
- net D7: now also U1.29 (GPIO18); no longer U1.9 (GPIO7)
- net D8: now also U1.28 (GPIO17); no longer U1.11 (GPIO8)
- net D9: now also U1.27 (GPIO16); no longer U1.12 (GPIO9)
- net LED_25: now also U1.2 (GPIO0); no longer U1.37 (GPIO25)

Commit message: Finish tracing
Connections:
- net D0: now also U1.14 (GPIO11); no longer U1.37 (GPIO25)
- net D1: now also U1.15 (GPIO12); no longer U1.36 (GPIO24)
- net D10: now also U1.32 (GPIO21); no longer U1.18 (GPIO15)
- net D11: now also U1.34 (GPIO22); no longer U1.17 (GPIO14)
- net D12: now also U1.35 (GPIO23); no longer U1.16 (GPIO13)
- net D13: now also U1.36 (GPIO24); no longer U1.15 (GPIO12)
- net D14: now also U1.37 (GPIO25); no longer U1.14 (GPIO11)
- net D2: now also U1.16 (GPIO13); no longer U1.35 (GPIO23)
- net D3: now also U1.17 (GPIO14); no longer U1.34 (GPIO22)
- net D4: now also U1.18 (GPIO15); no longer U1.32 (GPIO21)
- net D5: now also U1.27 (GPIO16); no longer U1.31 (GPIO20)
- net D6: now also U1.28 (GPIO17); no longer U1.30 (GPIO19)
- net D8: now also U1.30 (GPIO19); no longer U1.28 (GPIO17)
- net D9: now also U1.31 (GPIO20); no longer U1.27 (GPIO16)
Changed lines of the file:
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@@
 	(global_label "D1"
 		(shape bidirectional)
-		(at 104.14 110.49 0)
-		(fields_autoplaced yes)
-		(effects
-			(font
-				(size 1.27 1.27)
-			)
-			(justify left)
-		)
-		(property "Intersheetrefs" "${INTERSHEET_REFS}"
-			(at 110.716 110.49 0)
+		(at 104.14 80.01 0)
+		(fields_autoplaced yes)
+		(effects
+			(font
+				(size 1.27 1.27)
+			)
+			(justify left)
+		)
+		(property "Intersheetrefs" "${INTERSHEET_REFS}"
+			(at 110.716 80.01 0)
 			(effects
 				(font
@@
 	(global_label "D10"
 		(shape bidirectional)
-		(at 104.14 87.63 0)
-		(fields_autoplaced yes)
-		(effects
-			(font
-				(size 1.27 1.27)
-			)
-			(justify left)
-		)
-		(property "Intersheetrefs" "${INTERSHEET_REFS}"
-			(at 111.9255 87.63 0)
+		(at 104.14 102.87 0)
+		(fields_autoplaced yes)
+		(effects
+			(font
+				(size 1.27 1.27)
+			)
+			(justify left)
+		)
+		(property "Intersheetrefs" "${INTERSHEET_REFS}"
+			(at 111.9255 102.87 0)
 			(effects
 				(font
@@
 	(global_label "D0"
 		(shape bidirectional)
-		(at 104.14 113.03 0)
-		(fields_autoplaced yes)
-		(effects
-			(font
-				(size 1.27 1.27)
-			)
-			(justify left)
-		)
-		(property "Intersheetrefs" "${INTERSHEET_REFS}"
-			(at 110.716 113.03 0)
+		(at 104.14 77.47 0)
+		(fields_autoplaced yes)
+		(effects
+			(font
+				(size 1.27 1.27)
+			)
+			(justify left)
+		)
+		(property "Intersheetrefs" "${INTERSHEET_REFS}"
+			(at 110.716 77.47 0)
 			(effects
 				(font
@@
 	(global_label "D4"
 		(shape bidirectional)
-		(at 104.14 102.87 0)
-		(fields_autoplaced yes)
-		(effects
-			(font
-				(size 1.27 1.27)
-			)
-			(justify left)
-		)
-		(property "Intersheetrefs" "${INTERSHEET_REFS}"
-			(at 110.716 102.87 0)
+		(at 104.14 87.63 0)
+		(fields_autoplaced yes)
+		(effects
+			(font
+				(size 1.27 1.27)
+			)
+			(justify left)
+		)
+		(property "Intersheetrefs" "${INTERSHEET_REFS}"
+			(at 110.716 87.63 0)
 			(effects
 				(font
@@
 	(global_label "D8"
 		(shape bidirectional)
-		(at 104.14 92.71 0)
-		(fields_autoplaced yes)
-		(effects
-			(font
-				(size 1.27 1.27)
-			)
-			(justify left)
-		)
-		(property "Intersheetrefs" "${INTERSHEET_REFS}"
-			(at 110.716 92.71 0)
+		(at 104.14 97.79 0)
+		(fields_autoplaced yes)
+		(effects
+			(font
+				(size 1.27 1.27)
+			)
+			(justify left)
+		)
+		(property "Intersheetrefs" "${INTERSHEET_REFS}"
+			(at 110.716 97.79 0)
 			(effects
 				(font
@@
 	(global_label "D5"
 		(shape bidirectional)
-		(at 104.14 100.33 0)
-		(fields_autoplaced yes)
-		(effects
-			(font
-				(size 1.27 1.27)
-			)
-			(justify left)
-		)
-		(property "Intersheetrefs" "${INTERSHEET_REFS}"
-			(at 110.716 100.33 0)
+		(at 104.14 90.17 0)
+		(fields_autoplaced yes)
+		(effects
+			(font
+				(size 1.27 1.27)
+			)
+			(justify left)
+		)
+		(property "Intersheetrefs" "${INTERSHEET_REFS}"
+			(at 110.716 90.17 0)
 			(effects
 				(font
@@
 	(global_label "D6"
 		(shape bidirectional)
-		(at 104.14 97.79 0)
-		(fields_autoplaced yes)
-		(effects
-			(font
-				(size 1.27 1.27)
-			)
-			(justify left)
-		)
-		(property "Intersheetrefs" "${INTERSHEET_REFS}"
-			(at 110.716 97.79 0)
+		(at 104.14 92.71 0)
+		(fields_autoplaced yes)
+		(effects
+			(font
+				(size 1.27 1.27)
+			)
+			(justify left)
+		)
+		(property "Intersheetrefs" "${INTERSHEET_REFS}"
+			(at 110.716 92.71 0)
 			(effects
 				(font
@@
 	(global_label "D2"
 		(shape bidirectional)
-		(at 104.14 107.95 0)
-		(fields_autoplaced yes)
-		(effects
-			(font
-				(size 1.27 1.27)
-			)
-			(justify left)
-		)
-		(property "Intersheetrefs" "${INTERSHEET_REFS}"
-			(at 110.716 107.95 0)
+		(at 104.14 82.55 0)
+		(fields_autoplaced yes)
+		(effects
+			(font
+				(size 1.27 1.27)
+			)
+			(justify left)
+		)
+		(property "Intersheetrefs" "${INTERSHEET_REFS}"
+			(at 110.716 82.55 0)
 			(effects
 				(font
@@
 	(global_label "D13"
 		(shape bidirectional)
-		(at 104.14 80.01 0)
-		(fields_autoplaced yes)
-		(effects
-			(font
-				(size 1.27 1.27)
-			)
-			(justify left)
-		)
-		(property "Intersheetrefs" "${INTERSHEET_REFS}"
-			(at 111.9255 80.01 0)
+		(at 104.14 110.49 0)
+		(fields_autoplaced yes)
+		(effects
+			(font
+				(size 1.27 1.27)
+			)
+			(justify left)
+		)
+		(property "Intersheetrefs" "${INTERSHEET_REFS}"
+			(at 111.9255 110.49 0)
 			(effects
 				(font
@@
 	(global_label "D14"
 		(shape bidirectional)
-		(at 104.14 77.47 0)
-		(fields_autoplaced yes)
-		(effects
-			(font
-				(size 1.27 1.27)
-			)
-			(justify left)
-		)
-		(property "Intersheetrefs" "${INTERSHEET_REFS}"
-			(at 111.9255 77.47 0)
+		(at 104.14 113.03 0)
+		(fields_autoplaced yes)
+		(effects
+			(font
+				(size 1.27 1.27)
+			)
+			(justify left)
+		)
+		(property "Intersheetrefs" "${INTERSHEET_REFS}"
+			(at 111.9255 113.03 0)
 			(effects
 				(font
@@
 	(global_label "D3"
 		(shape bidirectional)
-		(at 104.14 105.41 0)
-		(fields_autoplaced yes)
-		(effects
-			(font
-				(size 1.27 1.27)
-			)
-			(justify left)
-		)
-		(property "Intersheetrefs" "${INTERSHEET_REFS}"
-			(at 110.716 105.41 0)
+		(at 104.14 85.09 0)
+		(fields_autoplaced yes)
+		(effects
+			(font
+				(size 1.27 1.27)
+			)
+			(justify left)
+		)
+		(property "Intersheetrefs" "${INTERSHEET_REFS}"
+			(at 110.716 85.09 0)
 			(effects
 				(font
@@
 	(global_label "D9"
 		(shape bidirectional)
-		(at 104.14 90.17 0)
-		(fields_autoplaced yes)
-		(effects
-			(font
-				(size 1.27 1.27)
-			)
-			(justify left)
-		)
-		(property "Intersheetrefs" "${INTERSHEET_REFS}"
-			(at 110.716 90.17 0)
+		(at 104.14 100.33 0)
+		(fields_autoplaced yes)
+		(effects
+			(font
+				(size 1.27 1.27)
+			)
+			(justify left)
+		)
+		(property "Intersheetrefs" "${INTERSHEET_REFS}"
+			(at 110.716 100.33 0)
 			(effects
 				(font
@@
 	(global_label "D11"
 		(shape bidirectional)
-		(at 104.14 85.09 0)
-		(fields_autoplaced yes)
-		(effects
-			(font
-				(size 1.27 1.27)
-			)
-			(justify left)
-		)
-		(property "Intersheetrefs" "${INTERSHEET_REFS}"
-			(at 111.9255 85.09 0)
+		(at 104.14 105.41 0)
+		(fields_autoplaced yes)
+		(effects
+			(font
+				(size 1.27 1.27)
+			)
+			(justify left)
+		)
+		(property "Intersheetrefs" "${INTERSHEET_REFS}"
+			(at 111.9255 105.41 0)
 			(effects
 				(font
@@
 	(global_label "D12"
 		(shape bidirectional)
-		(at 104.14 82.55 0)
-		(fields_autoplaced yes)
-		(effects
-			(font
-				(size 1.27 1.27)
-			)
-			(justify left)
-		)
-		(property "Intersheetrefs" "${INTERSHEET_REFS}"
-			(at 111.9255 82.55 0)
-			(effects
-				(font
+		(at 104.14 107.95 0)
+		(fields_autoplaced yes)
+		(effects
+			(font
+				(size 1.27 1.27)
+			)
+			(justify left)
+		)
+		(property "Intersheetrefs" "${INTERSHEET_REFS}"
+			(at 111.9255 107.95 0)
+			(effects
+				(font

Commit message: The finishing touches
Parts:
- J4: footprint Connector_USB:USB_A_Molex_48037-2200_Horizontal -> Connector_USB:USB_A_Keystone_931_Horizontal
Changed lines of the file:
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@@
 			)
 		)
-		(property "Footprint" "Connector_USB:USB_A_Molex_48037-2200_Horizontal"
+		(property "Footprint" "Connector_USB:USB_A_Keystone_931_Horizontal"
 			(at 40.64 163.83 0)
 			(effects

Commit message: Change USB port, adjust header position, start tracing
Parts:
- J4: footprint Connector_USB:USB_A_Keystone_931_Horizontal -> Connector_USB:USB_A_Onboard; LCSC C319178 -> (none); MPN 931 -> (none)
Changed lines of the file:
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@@
 			)
 		)
-		(property "Footprint" "Connector_USB:USB_A_Keystone_931_Horizontal"
+		(property "Footprint" "Connector_USB:USB_A_Onboard"
 			(at 40.64 163.83 0)
 			(effects
@@
 			)
 		)
-		(property "LCSC" "C319178"
+		(property "LCSC" ""
 			(at 36.83 162.56 0)
 			(effects
@@
 			)
 		)
-		(property "MPN" "931"
+		(property "MPN" ""
 			(at 36.83 162.56 0)
 			(effects

Commit message: Rev 2 of the Ragnohacks PCB
Parts:
- added J5: USB_C_Receptacle_USB2.0_16P, Connector_USB:USB_C_Receptacle_GCT_USB4105-xx-A_16P_TopMnt_Horizontal, symbol Connector:USB_C_Receptacle_USB2.0_16P
- added R5, R6: 5k1, Capacitor_SMD:C_0402_1005Metric, symbol Device:R
- J1: footprint Connector_PinHeader_2.54mm:PinHeader_1x02_P2.54mm_Vertical -> Connector_Wire:SolderWire-2sqmm_1x02_P7.8mm_D2mm_OD3.9mm
- J4: footprint Connector_USB:USB_A_Onboard -> Connector_USB:USB_A_Edge
Connections:
- net GND: now also J5.A1 (GND), J5.A12 (GND), J5.B1 (GND), J5.B12 (GND), J5.S1 (SHIELD), R5.1, R6.1
- net DN: now reaches J4.3 (D+), U4.1 (I/O1)
- net DN: now also J5.A7 (D-), J5.B7 (D-)
- net DP: now reaches J4.2 (D-), U4.3 (I/O2)
- net DP: now also J5.A6 (D+), J5.B6 (D+)
- net at D2.2 (A), J4.1 (VBUS): now also J5.A4 (VBUS), J5.A9 (VBUS), J5.B4 (VBUS), J5.B9 (VBUS)
- new net: J5.A5 (CC1), R5.2
- new net: J5.B5 (CC2), R6.2
- no-connect marks 0 -> 2
Other:
- moved on the sheet: C15, C17, C18, D1, D2, D3, J2, J3, J4, R3, R4, U2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
